File: SWITCHCONTROLLER.brd (EAGLE design)
At the start: 275 x 50 mm, 124 parts, among them IC1 MCP23017SO, IC2 MCP23017SO, IC3 MCP23017SO, IC4 MCP23017SO, IC5 MCP23017SO, IC6 MCP23017SO, J1 RJ45-X8, J2 RJ45-X8, J3 RJ45-X8, J5 M06-PIN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

Commit message: Added DC power jack and screw terminal
Parts:
- removed LED2: GREEN, SuperHouse-LEDs:LED-0603
- removed LED3: BLUE, SuperHouse-LEDs:LED3MM
- removed R39, R40: 2K2, SuperHouse-DiscreteSemi:R0603
- added D1: (no value), SuperHouse-DiscreteSemi:SMA-DIODE
- added J4: (no value), SuperHouse-Connectors:SCREWTERMINAL-3.5MM-2
- added J8: POWER_JACK-SLOTS, SuperHouse-Connectors:POWER_JACK_SLOTS
- LED1: device SuperHouse-LEDs:LED-0603 -> SuperHouse-LEDs:LED3MM
- moved LED1 58.0 mm to (55.0, 5.00), turned to 0 degrees
- moved R67 44.0 mm to (55.0, 9.00)
- moved J6 1.00 mm to (36.0, 7.00)
- moved J7 1.00 mm to (36.0, 39.0)
Connections:
- removed net N$7: LED1.A, R39.1
- removed net N$8: LED2.A, R40.1
- new net N$18: D1.A, J4.2, J8.PWR
- net GND: now also J4.1, J8.GND, J8.GNDBREAK, LED1.K; no longer LED1.C, LED2.C, LED3.K
- net N$13: now also LED1.A; no longer LED3.A
- net VCC: no longer R39.2, R67.2
- net VIN: now also D1.C, R67.2; no longer R40.2
Routing:
- net N$18: track 0.00 -> 43.2 mm
- net VCC: track 245.5 -> 231.3 mm
- net N$13: track 0.00 -> 4.21 mm
- net VIN: track 1.24 -> 4.32 mm, vias 1 -> 9
- net N$8: track 2.00 -> 0.00 mm
- net N$7: track 2.00 -> 0.00 mm
Other:
- board text added: "+"
- board text added: "-"
- board text added: "SKU: LSC24"
- board text added: "www.superhouse.tv/lsc24"
- board text removed: "SKU: I2CRJ45X8"
- board text removed: "www.superhouse.tv/switchcontroller"
