File: I2CRJ45X24.brd (EAGLE design)
At the start: 275 x 50 mm, 126 parts, among them IC1 MCP23017SO, IC2 MCP23017SO, IC3 MCP23017SO, IC4 MCP23017SO, IC5 MCP23017SO, IC6 MCP23017SO, J1 RJ45-X8, J2 RJ45-X8, J3 RJ45-X8, J4 POWER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

Commit message: Converted to I2C-BREAKOUT header for v2.0 release
Parts:
- added C7, C8: 330uF 50V, SuperHouse-DiscreteSemi:PANASONIC_G
- added J9: I2C-BREAKOUT, SuperHouse-Connectors:2X03-SHROUDED
- J5: value M06-PIN -> M01-PLAIN; device SuperHouse-Connectors:1X06-P -> SuperHouse-Connectors:1X01
- R67: value 1K5 -> 4K7
- moved J5 24.1 mm to (271.0, 16.0), turned to 0 degrees
Connections:
- new net !RESET: IC1.18, IC2.18, IC3.18, IC4.18, IC5.18, IC6.18, J9.6
- net !INT: now also J5.1; no longer J5.6
- net GND: now also C7.-, C8.-, J9.4; no longer J5.4
- net SCL: now also J9.1; no longer J5.2
- net SDA: now also J9.2; no longer J5.1
- net VCC: now also J9.5; no longer IC1.18, IC2.18, IC3.18, IC4.18, IC5.18, IC6.18, J5.3
- net VIN: now also C7.+, C8.+, J9.3; no longer J5.5
Routing:
- net !RESET: track 0.00 -> 245.8 mm, vias 0 -> 6
- net VCC: track 311.8 -> 283.3 mm
- net VIN: track 4.32 -> 19.8 mm, vias 9 -> 15
- net SDA: track 216.6 -> 230.8 mm
- net !INT: track 392.3 -> 379.0 mm
- net SCL: track 221.9 -> 228.3 mm
- net 3H6: track 30.6 -> 29.7 mm, vias 0 -> 1
Other:
- board text added: "!RST"
- board text added: "Copyright 2019-2020 SuperHouse Automation Pty Ltd Released under the terms of the TAPR Open Hardware License: www.tapr.org/OHL"
- board text added: "I2C-BREAKOUT"
- board text added: "v2.0"
- board text removed: "Copyright 2019 SuperHouse Automation Pty Ltd Released under the terms of the TAPR Open Hardware License: www.tapr.org/OHL"
- board text removed: "v1.0"

Commit message: Moved holes back from edge for v2.1 release
Routing:
- net !INT: track 379.0 -> 382.0 mm
Other:
- board text added: "v2.1"
- board text removed: "v2.0"
Changed lines of the file:
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@@
 </layers>
 <board>
-<fusionsync huburn="a.cGVyc29uYWw6dWUyZDliZmNi" projecturn="a.cGVyc29uYWw6dWUyZDliZmNiIzIwMTkwNjE5MTk5NjgzNjgx" f3durn="urn:adsk.wipprod:dm.lineage:7PE12rU6Rs2d8xNWJ3I8mw" pcbguid="240f1cde-c83f-4e3e-9fac-562d2bf45fdf" lastpulledtime="" lastsyncedchangeguid="1491f9b9-a179-9c0a-9821-19275fe4b9b0" latestrevisionid="" lastsyncedrevisionid="" lastboardhashguid="0d0417fb-bed7-953d-fd56-26c786d4b7d5" lastpushedtime="2020-04-07T05:19:51Z" linktopcb3d="%12"/>
+<fusionsync huburn="a.cGVyc29uYWw6dWUyZDliZmNi" projecturn="a.cGVyc29uYWw6dWUyZDliZmNiIzIwMTkwNjE5MTk5NjgzNjgx" f3durn="urn:adsk.wipprod:dm.lineage:7PE12rU6Rs2d8xNWJ3I8mw" pcbguid="240f1cde-c83f-4e3e-9fac-562d2bf45fdf" lastpulledtime="" lastsyncedchangeguid="1491f9b9-a179-9c0a-9821-19275fe4b9b0" latestrevisionid="" lastsyncedrevisionid="" lastboardhashguid="9dd74273-d936-b2ac-470b-90bfb06084ef" lastpushedtime="2020-04-13T07:39:58Z" linktopcb3d="%12"/>
 <plain>
 <wire x1="3" y1="0" x2="0" y2="3" width="0" layer="20" curve="-90"/>
@@
 <wire x1="275" y1="3" x2="272" y2="0" width="0" layer="20" curve="-90"/>
 <wire x1="272" y1="0" x2="3" y2="0" width="0" layer="20"/>
-<text x="6.953" y="46.623" size="1.778" layer="21" font="vector" ratio="17">v2.0</text>
+<text x="6.953" y="46.623" size="1.778" layer="21" font="vector" ratio="17">v2.1</text>
 <text x="95.455" y="46.854" size="2.1844" layer="21" font="vector" ratio="17" align="bottom-center">www.superhouse.tv/i2crj45x24</text>
 <text x="162.191" y="47.171" size="1.27" layer="21" font="vector" ratio="17">SKU: I2CRJ45X24</text>
-<hole x="3" y="3" drill="3.2"/>
-<hole x="202" y="3" drill="3.2"/>
+<hole x="3" y="8" drill="3.2"/>
+<hole x="202" y="8" drill="3.2"/>
 <hole x="202" y="47" drill="3.2"/>
 <hole x="3" y="47" drill="3.2"/>
-<hole x="132" y="3" drill="3.2"/>
+<hole x="132" y="8" drill="3.2"/>
 <text x="81.191" y="45.171" size="1.27" layer="21" font="vector" ratio="17" align="bottom-center">0x20</text>
 <text x="113.191" y="45.171" size="1.27" layer="21" font="vector" ratio="17" align="bottom-center">0x21</text>
@@
 <text x="12.455" y="32.854" size="3.1" layer="21" font="vector" ratio="17" distance="30" align="center-left">Super
 House</text>
-<text x="2.455" y="14.854" size="2.8" layer="21" font="vector" ratio="17" distance="30">24 Channel
+<text x="2.455" y="16" size="2.8" layer="21" font="vector" ratio="17" distance="20">24 Channel
 I2C RJ45
 Breakout</text>
-<text x="4.5" y="12.6" size="1.4224" layer="21" font="vector" ratio="17" distance="30">by Jon Oxer</text>
+<text x="9.5" y="14.2" size="1.4224" layer="21" font="vector" ratio="17" distance="30">by Jon Oxer</text>
 <text x="193.455" y="32.854" size="1.6764" layer="22" font="vector" ratio="17" distance="30" rot="MR0">Copyright 2019-2020 SuperHouse Automation Pty Ltd
 Released under the terms
@@
 <text x="177.691" y="25.171" size="1.27" layer="21" font="vector" ratio="17">MCP23017</text>
 <circle x="3" y="47" radius="3.201559375" width="0.254" layer="41"/>
-<circle x="3" y="3" radius="3.201559375" width="0.254" layer="41"/>
-<circle x="132" y="3" radius="3.201559375" width="0.254" layer="41"/>
-<circle x="202" y="3" radius="3.201559375" width="0.254" layer="41"/>
+<circle x="3" y="8" radius="3.201559375" width="0.254" layer="41"/>
+<circle x="132" y="8" radius="3.201559375" width="0.254" layer="41"/>
+<circle x="202" y="8" radius="3.201559375" width="0.254" layer="41"/>
 <circle x="202" y="47" radius="3.201559375" width="0.254" layer="41"/>
 <circle x="132" y="47" radius="3.201559375" width="0.254" layer="41"/>
@@
 <circle x="132" y="47" radius="3.201559375" width="0.254" layer="42"/>
 <circle x="202" y="47" radius="3.201559375" width="0.254" layer="42"/>
-<circle x="132" y="3" radius="3.201559375" width="0.254" layer="42"/>
-<circle x="202" y="3" radius="3.201559375" width="0.254" layer="42"/>
-<circle x="3" y="3" radius="3.201559375" width="0.254" layer="42"/>
-<circle x="62" y="3" radius="3.201559375" width="0.254" layer="42"/>
-<circle x="62" y="3" radius="3.201559375" width="0.254" layer="41"/>
-<hole x="62" y="3" drill="3.2"/>
-<circle x="272" y="3" radius="3.201559375" width="0.254" layer="42"/>
-<circle x="272" y="3" radius="3.201559375" width="0.254" layer="41"/>
-<hole x="272" y="3" drill="3.2"/>
+<circle x="132" y="8" radius="3.201559375" width="0.254" layer="42"/>
+<circle x="202" y="8" radius="3.201559375" width="0.254" layer="42"/>
+<circle x="3" y="8" radius="3.201559375" width="0.254" layer="42"/>
+<circle x="62" y="8" radius="3.201559375" width="0.254" layer="42"/>
+<circle x="62" y="8" radius="3.201559375" width="0.254" layer="41"/>
+<hole x="62" y="8" drill="3.2"/>
+<circle x="272" y="8" radius="3.201559375" width="0.254" layer="42"/>
+<circle x="272" y="8" radius="3.201559375" width="0.254" layer="41"/>
+<hole x="272" y="8" drill="3.2"/>
 <text x="221.191" y="45.171" size="1.27" layer="21" font="vector" ratio="17" align="bottom-center">0x24</text>
 <text x="253.191" y="45.171" size="1.27" layer="21" font="vector" ratio="17" align="bottom-center">0x25</text>
@@
 <dimension x1="275" y1="51" x2="272" y2="51" x3="273.5" y3="54" textsize="1.778" layer="47"/>
 <dimension x1="0" y1="51" x2="3" y2="51" x3="1.5" y3="54" textsize="1.778" layer="47"/>
-<dimension x1="-1" y1="3" x2="-1" y2="47" x3="-2" y3="25" textsize="1.778" layer="47"/>
-<dimension x1="-1" y1="0" x2="-1" y2="3" x3="-5" y3="1.5" textsize="1.778" layer="47"/>
+<dimension x1="-1" y1="8" x2="-1" y2="47" x3="-2" y3="27.5" textsize="1.778" layer="47"/>
+<dimension x1="-1" y1="0" x2="-1" y2="8" x3="-5" y3="4" textsize="1.778" layer="47"/>
 <dimension x1="-1" y1="50" x2="-1" y2="47" x3="-5" y3="48.5" textsize="1.778" layer="47"/>
 <rectangle x1="20" y1="3" x2="26" y2="8" layer="1"/>
@@
 <text x="22.5" y="47" size="3.81" layer="21" font="vector" ratio="16" align="center">-</text>
 <text x="52" y="5" size="0.8128" layer="21" font="vector" ratio="12">A</text>
-<text x="4.455" y="6.354" size="1.8" layer="21" font="vector" ratio="17" distance="30" align="bottom-center">12Vdc</text>
+<text x="4.455" y="2.354" size="1.8" layer="21" font="vector" ratio="17" distance="30" align="bottom-center">12Vdc</text>
 <text x="16.146" y="43.455" size="1.9304" layer="21" font="vector" ratio="17" distance="30" rot="R90" align="bottom-center">12Vdc</text>
 <text x="50" y="19" size="1.6764" layer="21" font="vector" ratio="12">1: Data 1
@@
 <text x="47" y="13" size="1.27" layer="21" font="vector" ratio="12">1K in series with
 each data line</text>
-<circle x="4" y="10" radius="0.3" width="0.4" layer="21"/>
-<wire x1="3.5" y1="11" x2="3.5" y2="9" width="0.4" layer="21" curve="-233.130102"/>
-<wire x1="4" y1="10" x2="2" y2="10" width="0.254" layer="21"/>
-<wire x1="5.2" y1="10" x2="6.5" y2="10" width="0.254" layer="21"/>
-<wire x1="6" y1="11" x2="7" y2="11" width="0.254" layer="21"/>
-<wire x1="2" y1="10.5" x2="2" y2="11.5" width="0.254" layer="21"/>
-<wire x1="2.5" y1="11" x2="1.5" y2="11" width="0.254" layer="21"/>
+<circle x="4" y="13" radius="0.3" width="0.4" layer="21"/>
+<wire x1="3.5" y1="14" x2="3.5" y2="12" width="0.4" layer="21" curve="-233.130102"/>
+<wire x1="4" y1="13" x2="2" y2="13" width="0.254" layer="21"/>
+<wire x1="5.2" y1="13" x2="6.5" y2="13" width="0.254" layer="21"/>
+<wire x1="6" y1="14" x2="7" y2="14" width="0.254" layer="21"/>
+<wire x1="2" y1="13.5" x2="2" y2="14.5" width="0.254" layer="21"/>
+<wire x1="2.5" y1="14" x2="1.5" y2="14" width="0.254" layer="21"/>
 <text x="264.191" y="36.551" size="1.016" layer="22" font="vector" ratio="17" rot="MR0" align="center-right">!RST</text>
 <text x="259.809" y="42.529" size="1.4224" layer="21" font="vector" ratio="17" rot="R180" align="center-right">I2C-BREAKOUT</text>
@@
 <wire x1="250.46" y1="37.54" x2="248.22" y2="37.54" width="0.254" layer="1"/>
 <wire x1="251" y1="12" x2="253" y2="10" width="0.254" layer="1"/>
-<wire x1="253" y1="10" x2="269" y2="10" width="0.254" layer="1"/>
-<wire x1="269" y1="10" x2="271" y2="12" width="0.254" layer="1"/>
+<wire x1="253" y1="10" x2="267" y2="10" width="0.254" layer="1"/>
+<wire x1="267" y1="10" x2="271" y2="14" width="0.254" layer="1"/>
 <via x="222" y="9" extent="1-16" drill="0.5"/>
 <via x="248" y="9" extent="1-16" drill="0.5"/>
@@
 <wire x1="217" y1="10" x2="218" y2="9" width="0.254" layer="16"/>
 <wire x1="218" y1="9" x2="222" y2="9" width="0.254" layer="16"/>
-<wire x1="189" y1="10" x2="217" y2="10" width="0.254" layer="16"/>
+<wire x1="189" y1="10" x2="197" y2="10" width="0.254" layer="16"/>
+<wire x1="197" y1="10" x2="200" y2="13" width="0.254" layer="16"/>
+<wire x1="200" y1="13" x2="204" y2="13" width="0.254" layer="16"/>
+<wire x1="204" y1="13" x2="207" y2="10" width="0.254" layer="16"/>
+<wire x1="207" y1="10" x2="217" y2="10" width="0.254" layer="16"/>
 <via x="85" y="9" extent="1-16" drill="0.5"/>
 <wire x1="85" y1="9" x2="108" y2="9" width="0.254" layer="16"/>
@@
 <wire x1="108" y1="9" x2="111" y2="12" width="0.254" layer="1"/>
 <contactref element="J5" pad="1"/>
-<wire x1="271" y1="12" x2="271" y2="16" width="0.254" layer="1"/>
-<wire x1="112.006328125" y1="10.993671875" x2="150.993671875" y2="10.993671875" width="0.254" layer="1"/>
+<wire x1="271" y1="14" x2="271" y2="16" width="0.254" layer="1"/>
+<wire x1="112.006328125" y1="10.993671875" x2="127.993671875" y2="10.993671875" width="0.254" layer="1"/>
+<wire x1="127.993671875" y1="10.993671875" x2="130" y2="13" width="0.254" layer="1"/>
+<wire x1="130" y1="13" x2="134" y2="13" width="0.254" layer="1"/>
+<wire x1="134" y1="13" x2="136" y2="11" width="0.254" layer="1"/>
+<wire x1="136" y1="11" x2="150.993671875" y2="10.993671875" width="0.254" layer="1"/>
 </signal>
 <signal name="2A1">

Commit message: Removed Ethernet passthrough and shortened board.
Parts:
- removed D1: SS56, SuperHouse-DiscreteSemi:SMA-DIODE
- removed J6, J7: RJ45-X1-METAL, SuperHouse-Connectors:RJ45-1X1
- removed J8: POWER_JACK-SLOTS, SuperHouse-Connectors:POWER_JACK_SLOTS
- removed LED1: BLUE, SuperHouse-LEDs:LED3MM
- removed R67: 4K7, SuperHouse-DiscreteSemi:R0603
- added LED2: BLUE, SuperHouse-LEDs:LED-0603
- added LED3: GREEN, SuperHouse-LEDs:LED-0603
- added R39, R40: 2K2, SuperHouse-DiscreteSemi:R0603
- J4: value POWER -> I2C-BREAKOUT; device SuperHouse-Connectors:SCREWTERMINAL-3.5MM-2 -> SuperHouse-Connectors:2X03-SHROUDED
- moved J5 61.0 mm to (211.5, 2.50)
- moved C1 59.0 mm to (30.0, 45.0)
- moved C2 59.0 mm to (62.0, 45.0)
- moved C3 59.0 mm to (100.0, 45.0)
- moved C4 59.0 mm to (123.5, 48.0)
- moved C5 59.0 mm to (162.0, 48.0)
- moved C6 59.0 mm to (194.0, 48.0)
- moved C7 59.0 mm to (73.0, 31.0)
- moved C8 59.0 mm to (143.0, 31.0)
- moved FID2 59.0 mm to (197.5, 6.00)
- moved FID3 59.0 mm to (55.0, 31.5)
- moved IC1 59.0 mm to (22.0, 35.0)
- moved IC2 59.0 mm to (54.0, 35.0)
- moved IC3 59.0 mm to (92.0, 35.0)
- moved IC4 59.0 mm to (124.0, 35.0)
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Connections:
- removed net N$10: J6.6, J7.6
- removed net N$11: J6.7, J7.7
- removed net N$12: J6.8, J7.8
- removed net N$13: LED1.A, R67.1
- removed net N$18: D1.A, J4.2, J8.PWR
- removed net N$3: J6.1, J7.1
- removed net N$4: J6.2, J7.2
- removed net N$5: J6.3, J7.3
- removed net N$6: J6.4, J7.4
- removed net N$9: J6.5, J7.5
- new net N$7: LED2.A, R39.1
- new net N$8: LED3.A, R40.1
- net !RESET: now also J4.6
- net GND: now also J4.4, LED2.C, LED3.C; no longer J4.1, J8.GND, J8.GNDBREAK, LED1.K
- net SCL: now also J4.1
- net SDA: now also J4.2
- net VCC: now also J4.5, R39.2
- net VIN: now also J4.3, R40.2; no longer D1.C, R67.2
Routing:
- net VCC: track 283.3 -> 332.3 mm, vias 2 -> 3
- net N$18: track 43.2 -> 0.00 mm
- net N$12: track 43.1 -> 0.00 mm
- net N$3: track 40.1 -> 0.00 mm
- net N$11: track 39.4 -> 0.00 mm
- net N$5: track 34.8 -> 0.00 mm
- net N$10: track 30.4 -> 0.00 mm
- net N$9: track 28.2 -> 0.00 mm
- net SDA: track 230.8 -> 256.6 mm, vias 7 -> 8
- net SCL: track 228.3 -> 253.7 mm
- net N$4: track 23.9 -> 0.00 mm
- net N$6: track 21.7 -> 0.00 mm
- net !RESET: track 245.8 -> 264.5 mm
- net !INT: track 382.0 -> 387.0 mm
- net N$13: track 4.21 -> 0.00 mm
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Other:
- board size 275 x 50 mm -> 216 x 50 mm
- board text added: "Copyright 2019-2021 SuperHouse Automation Pty Ltd Released under the terms of the TAPR Open Hardware License: www.tapr.org/OHL"
- board text added: "v2.2"
- board text removed: "+"
- board text removed: "-"
- board text removed: "12Vdc"
- board text removed: "A"
- board text removed: "Copyright 2019-2020 SuperHouse Automation Pty Ltd Released under the terms of the TAPR Open Hardware License: www.tapr.org/OHL"
- board text removed: "Ethernet Pass- through"
- board text removed: "v2.1"
