File: Hardware/I2CRJ45X24.sch (EAGLE design)
At the start: 97 parts, among them IC1 MCP23017SO, IC2 MCP23017SO, IC3 MCP23017SO, IC4 MCP23017SO, IC5 MCP23017SO, IC6 MCP23017SO, J1 I2C-BREAKOUT, J2 I2C-BREAKOUT, J3 M01-PLAIN, J4 RJ45-X8, J5 RJ45-X8, J6 RJ45-X8

Commit message: Replace discrete resistors with resistor networks. Add hardware pull-ups to all input lines. Routing, ERC, and DRC for v3.0 release.
Parts:
- removed R39, R40, R67, R68, R69, R70, R71, R72, R73, R74, R75, R76, R77, R78, R79, R80, R81, R82, R83, R84, R85, R86, R87, R88, R89, R90, R91, R92, R93, R94, R95, R96: 1K, SuperHouse-DiscreteSemi:RESISTOR0603
- added C9: 330uF 50V, SuperHouse-Capacitors:CAP_POLG
- added RN33, RN34, RN35, RN36, RN37, RN38, RN39, RN40: 1K, SuperHouse-Resistors:4R-NCAY16
- added RN41, RN42, RN43, RN44, RN45, RN46, RN47, RN48: 10K, SuperHouse-Resistors:4R-NCAY16
- C1, C2, C3, C4, C5, C6: device SuperHouse-DiscreteSemi:CAP0805 -> SuperHouse-Capacitors:CAP0805
- C7, C8: device SuperHouse-DiscreteSemi:CAP_POLG -> SuperHouse-Capacitors:CAP_POLG
- R100, R101, R97, R98, R99: device SuperHouse-DiscreteSemi:RESISTOR0603 -> SuperHouse-Resistors:RESISTOR0603
- RN1, RN10, RN11, RN12, RN13, RN14, RN15, RN16, RN17, RN18, RN19, RN2, RN20, RN21, RN22, RN23, RN24, RN25, RN26, RN27, RN28, RN29, RN3, RN30, RN31, RN32, RN4, RN5, RN6, RN7, RN8, RN9: device SuperHouse-DiscreteSemi:4R-NCAY16 -> SuperHouse-Resistors:4R-NCAY16
Connections:
- net 3A1: now also RN33D.2, RN44D.1; no longer R70.2
- net 3A2: now also RN33C.2, RN44C.1; no longer R72.2
- net 3A3: now also RN33B.2, RN44B.1; no longer R71.2
- net 3A6: now also RN33A.2, RN44A.1; no longer R73.2
- net 3B1: now also RN35D.2, RN42D.1; no longer R84.2
- net 3B2: now also RN35C.2, RN42C.1; no longer R82.2
- net 3B3: now also RN35B.2, RN42B.1; no longer R80.2
- net 3B6: now also RN35A.2, RN42A.1; no longer R78.2
- net 3C1: now also RN37D.2, RN48D.1; no longer R86.2
- net 3C2: now also RN37C.2, RN48C.1; no longer R88.2
- net 3C3: now also RN37B.2, RN48B.1; no longer R87.2
- net 3C6: now also RN37A.2, RN48A.1; no longer R89.2
- net 3D1: now also RN39D.2, RN46D.1; no longer R68.2
- net 3D2: now also RN39C.2, RN46C.1; no longer R40.2
- net 3D3: now also RN39B.2, RN46B.1; no longer R96.2
- net 3D6: now also RN39A.2, RN46A.1; no longer R94.2
- net 3E1: now also RN34D.2, RN43D.1; no longer R76.2
- net 3E2: now also RN34C.2, RN43C.1; no longer R75.2
- net 3E3: now also RN34B.2, RN43B.1; no longer R74.2
- net 3E6: now also RN34A.2, RN43A.1; no longer R77.2
- net 3F1: now also RN36D.2, RN41D.1; no longer R85.2
- net 3F2: now also RN36C.2, RN41C.1; no longer R83.2
- net 3F3: now also RN36B.2, RN41B.1; no longer R81.2
- net 3F6: now also RN36A.2, RN41A.1; no longer R79.2
- net 3G1: now also RN38D.2, RN47D.1; no longer R92.2
- net 3G2: now also RN38C.2, RN47C.1; no longer R91.2
- net 3G3: now also RN38B.2, RN47B.1; no longer R90.2
- net 3G6: now also RN38A.2, RN47A.1; no longer R93.2
- net 3H1: now also RN40D.2, RN45D.1; no longer R67.2
- net 3H2: now also RN40C.2, RN45C.1; no longer R69.2
- net 3H3: now also RN40B.2, RN45B.1; no longer R39.2
- net 3H6: now also RN40A.2, RN45A.1; no longer R95.2
- net GND: now also C9.-
- net GPA0-5: now also RN33D.1; no longer R70.1
- net GPA0-6: now also RN37D.1; no longer R86.1
- net GPA1-5: now also RN33C.1; no longer R72.1
- net GPA1-6: now also RN37C.1; no longer R88.1
- net GPA2-5: now also RN33B.1; no longer R71.1
- net GPA2-6: now also RN37B.1; no longer R87.1
- net GPA3-5: now also RN33A.1; no longer R73.1
- net GPA3-6: now also RN37A.1; no longer R89.1
- net GPA4-5: now also RN34D.1; no longer R76.1
- net GPA4-6: now also RN38D.1; no longer R92.1
- net GPA5-5: now also RN34C.1; no longer R75.1
- net GPA5-6: now also RN38C.1; no longer R91.1
- net GPA6-5: now also RN34B.1; no longer R74.1
- net GPA6-6: now also RN38B.1; no longer R90.1
- net GPA7-5: now also RN34A.1; no longer R77.1
- net GPA7-6: now also RN38A.1; no longer R93.1
- net GPB0-5: now also RN35D.1; no longer R84.1
- net GPB0-6: now also RN39D.1; no longer R68.1
- net GPB1-5: now also RN35C.1; no longer R82.1
- net GPB1-6: now also RN39C.1; no longer R40.1
- net GPB2-5: now also RN35B.1; no longer R80.1
- net GPB2-6: now also RN39B.1; no longer R96.1
- net GPB3-5: now also RN35A.1; no longer R78.1
- net GPB3-6: now also RN39A.1; no longer R94.1
- net GPB4-5: now also RN36D.1; no longer R85.1
- net GPB4-6: now also RN40D.1; no longer R67.1
- net GPB5-5: now also RN36C.1; no longer R83.1
- net GPB5-6: now also RN40C.1; no longer R69.1
- net GPB6-5: now also RN36B.1; no longer R81.1
- net GPB6-6: now also RN40B.1; no longer R39.1
- net GPB7-5: now also RN36A.1; no longer R79.1
- net GPB7-6: now also RN40A.1; no longer R95.1
- net VCC: now also RN41A.2, RN41B.2, RN41C.2, RN41D.2, RN42A.2, RN42B.2, RN42C.2, RN42D.2, RN43A.2, RN43B.2, RN43C.2, RN43D.2, RN44A.2, RN44B.2, RN44C.2, RN44D.2, RN45A.2, RN45B.2, RN45C.2, RN45D.2, RN46A.2, RN46B.2, RN46C.2, RN46D.2, RN47A.2, RN47B.2, RN47C.2, RN47D.2, RN48A.2, RN48B.2, RN48C.2, RN48D.2
- net VIN: now also C9.+
Other:
- note added: "V3.0 (2021-06-04)"
- note removed: "V3.0 (2021-04-15)"
