File: Hardware/I2CRJ45X8.sch (EAGLE design)
At the start: 65 parts, among them IC1 MCP23017SO, IC2 MCP23017SO, J1 I2C-BREAKOUT, J2 I2C-BREAKOUT, J3 M01-PLAIN, J4 RJ45-X8

Commit message: Regenerated 8-port version from updated 16-port version.
Parts:
- removed R1, R10, R11, R12, R13, R14, R15, R16, R17, R18, R19, R2, R20, R21, R22, R23, R24, R25, R26, R27, R28, R29, R3, R30, R31, R32, R4, R5, R6, R7, R8, R9: 1K, SuperHouse-DiscreteSemi:RESISTOR0603
- removed R33, R34, R35, R36: 4K7, SuperHouse-DiscreteSemi:RESISTOR0603
- removed R37, R38, R39, R40, R41, R42, R43: 10K, SuperHouse-DiscreteSemi:RESISTOR0603
- removed SJ4, SJ7: A0, SuperHouse-Jumpers:SJ-NORMAL
- removed SJ5, SJ8: A1, SuperHouse-Jumpers:SJ-NORMAL
- removed SJ6, SJ9: A2, SuperHouse-Jumpers:SJ-NORMAL
- added C7: 330uF 50V, SuperHouse-Capacitors:CAP_POLG
- added J12: I2C Addr 2, SuperHouse-Connectors:M02X3-PIN
- added J7: I2C Addr 1, SuperHouse-Connectors:M02X3-PIN
- added R100, R97, R98, R99: 4K7, SuperHouse-Resistors:RESISTOR0603
- added R101: 10K, SuperHouse-Resistors:RESISTOR0603
- added RN1, RN10, RN11, RN12, RN2, RN3, RN4, RN9: 1K, SuperHouse-Resistors:4R-NCAY16
- added RN13, RN14, RN15, RN16, RN49, RN5, RN50, RN6, RN7, RN8: 10K, SuperHouse-Resistors:4R-NCAY16
- C1, C2: device SuperHouse-DiscreteSemi:CAP0805 -> SuperHouse-Capacitors:CAP0805
- SJ1, SJ2: device SuperHouse-Jumpers:SJ-NORMAL -> SuperHouse-Connectors:M02-PIN
Connections:
- net !RESET: now also R101.1; no longer R39.1
- net 1A1: now also RN1D.2, RN5D.1; no longer R1.2
- net 1A2: now also RN1C.2, RN5C.1; no longer R3.2
- net 1A3: now also RN1B.2, RN5B.1; no longer R2.2
- net 1A6: now also RN1A.2, RN5A.1; no longer R4.2
- net 1B1: now also RN3D.2, RN7D.1; no longer R15.2
- net 1B2: now also RN3C.2, RN7C.1; no longer R13.2
- net 1B3: now also RN3B.2, RN7B.1; no longer R11.2
- net 1B6: now also RN3A.2, RN7A.1; no longer R9.2
- net 1C1: now also RN13D.1, RN9D.2; no longer R17.2
- net 1C2: now also RN13C.1, RN9C.2; no longer R19.2
- net 1C3: now also RN13B.1, RN9B.2; no longer R18.2
- net 1C6: now also RN13A.1, RN9A.2; no longer R20.2
- net 1D1: now also RN11D.2, RN15D.1; no longer R31.2
- net 1D2: now also RN11C.2, RN15C.1; no longer R29.2
- net 1D3: now also RN11B.2, RN15B.1; no longer R27.2
- net 1D6: now also RN11A.2, RN15A.1; no longer R25.2
- net 1E1: now also RN2D.2, RN6D.1; no longer R7.2
- net 1E2: now also RN2C.2, RN6C.1; no longer R6.2
- net 1E3: now also RN2B.2, RN6B.1; no longer R5.2
- net 1E6: now also RN2A.2, RN6A.1; no longer R8.2
- net 1F1: now also RN4D.2, RN8D.1; no longer R16.2
- net 1F2: now also RN4C.2, RN8C.1; no longer R14.2
- net 1F3: now also RN4B.2, RN8B.1; no longer R12.2
- net 1F6: now also RN4A.2, RN8A.1; no longer R10.2
- net 1G1: now also RN10D.2, RN14D.1; no longer R23.2
- net 1G2: now also RN10C.2, RN14C.1; no longer R22.2
- net 1G3: now also RN10B.2, RN14B.1; no longer R21.2
- net 1G6: now also RN10A.2, RN14A.1; no longer R24.2
- net 1H1: now also RN12D.2, RN16D.1; no longer R32.2
- net 1H2: now also RN12C.2, RN16C.1; no longer R30.2
- net 1H3: now also RN12B.2, RN16B.1; no longer R28.2
- net 1H6: now also RN12A.2, RN16A.1; no longer R26.2
- net GND: now also C7.-, RN49A.1, RN49B.1, RN49C.1, RN49D.1, RN50A.1, RN50B.1, RN50C.1, RN50D.1; no longer R37.1, R38.1, R40.1, R41.1, R42.1, R43.1
- net GPA0-1: now also RN1D.1; no longer R1.1
- net GPA0-2: now also RN9D.1; no longer R17.1
- net GPA1-1: now also RN1C.1; no longer R3.1
- net GPA1-2: now also RN9C.1; no longer R19.1
- net GPA2-1: now also RN1B.1; no longer R2.1
- net GPA2-2: now also RN9B.1; no longer R18.1
- net GPA3-1: now also RN1A.1; no longer R4.1
- net GPA3-2: now also RN9A.1; no longer R20.1
- net GPA4-1: now also RN2D.1; no longer R7.1
- net GPA4-2: now also RN10D.1; no longer R23.1
- net GPA5-1: now also RN2C.1; no longer R6.1
- net GPA5-2: now also RN10C.1; no longer R22.1
- net GPA6-1: now also RN2B.1; no longer R5.1
- net GPA6-2: now also RN10B.1; no longer R21.1
- net GPA7-1: now also RN2A.1; no longer R8.1
- net GPA7-2: now also RN10A.1; no longer R24.1
- net GPB0-1: now also RN3D.1; no longer R15.1
- net GPB0-2: now also RN11D.1; no longer R31.1
- net GPB1-1: now also RN3C.1; no longer R13.1
- net GPB1-2: now also RN11C.1; no longer R29.1
- net GPB2-1: now also RN3B.1; no longer R11.1
- net GPB2-2: now also RN11B.1; no longer R27.1
- net GPB3-1: now also RN3A.1; no longer R9.1
- net GPB3-2: now also RN11A.1; no longer R25.1
- net GPB4-1: now also RN4D.1; no longer R16.1
- net GPB4-2: now also RN12D.1; no longer R32.1
- net GPB5-1: now also RN4C.1; no longer R14.1
- net GPB5-2: now also RN12C.1; no longer R30.1
- net GPB6-1: now also RN4B.1; no longer R12.1
- net GPB6-2: now also RN12B.1; no longer R28.1
- net GPB7-1: now also RN4A.1; no longer R10.1
- net GPB7-2: now also RN12A.1; no longer R26.1
- net N$1: now also R99.2; no longer R35.2
- net N$10: now also J12.4, RN50B.2; no longer R37.2, SJ8.1
- net N$11: now also IC2.A2, J12.6, RN50A.2; no longer IC2.A0, R43.2, SJ7.1
- net N$2: now also R100.2; no longer R36.2
- net N$3: now also R101.2; no longer R39.2
- net N$4: now also J7.6, RN49A.2; no longer R42.2, SJ6.1
- net N$5: now also J7.4, RN49B.2; no longer R41.2, SJ5.1
- net N$6: now also J7.2, RN49C.2; no longer R40.2, SJ4.1
- net N$7: now also R97.1; no longer R33.1
- net N$8: now also R98.1; no longer R34.1
- net N$9: now also IC2.A0, J12.2, RN50C.2; no longer IC2.A2, R38.2, SJ9.1
- net SCL: now also R99.1; no longer R35.1
- net SDA: now also R100.1; no longer R36.1
- net VCC: now also J12.1, J12.3, J12.5, J7.1, J7.3, J7.5, R97.2, RN13A.2, RN13B.2, RN13C.2, RN13D.2, RN14A.2, RN14B.2, RN14C.2, RN14D.2, RN15A.2, RN15B.2, RN15C.2, RN15D.2, RN16A.2, RN16B.2, RN16C.2, RN16D.2, RN5A.2, RN5B.2, RN5C.2, RN5D.2, RN6A.2, RN6B.2, RN6C.2, RN6D.2, RN7A.2, RN7B.2, RN7C.2, RN7D.2, RN8A.2, RN8B.2, RN8C.2, RN8D.2; no longer R33.2, SJ4.2, SJ5.2, SJ6.2, SJ7.2, SJ8.2, SJ9.2
- net VIN: now also C7.+, R98.2; no longer R34.2
Other:
- note added: "I2C Addr: 0x20 - 0x27"
- note added: "I2C Addresses: 0x20-0x27"
- note added: "V3.0 (2021-06-08)"
- note removed: "I2C Addr: 0x20"
- note removed: "I2C Addresses: 0x20-0x25"
- note removed: "V3.0 (2021-04-15)"
